File: Eagle/ZX81KBD/zx81_kbd v0.4.brd (EAGLE design)
At the start: 99.1 x 82.5 mm, 119 parts, among them IC1 REG1117, IC3 PCF8574P

Commit message: Initial public version
Parts:
- moved JP2 2.54 mm to (16.1, 43.2)
- moved S1 0.25 mm to (-27.9, 77.7)
- moved S2 0.25 mm to (-15.2, 77.7)
Routing:
- net VCC: track 334.3 -> 340.3 mm
- net GND: track 438.1 -> 443.4 mm
- net MISO: track 96.1 -> 98.8 mm
- net SCK: track 129.1 -> 131.6 mm
- net /RFSH: track 83.6 -> 81.4 mm
- net /ROMCS: track 74.1 -> 76.0 mm
- net N$38: track 56.3 -> 58.1 mm
- net A4: track 73.7 -> 75.3 mm
- net /M1: track 88.4 -> 90.0 mm
- net MOSI: track 97.8 -> 99.1 mm
- net D7: track 143.8 -> 144.6 mm
- net N$37: track 98.7 -> 99.2 mm
Other:
- board size 99.1 x 82.5 mm -> 100.5 x 82.5 mm

Commit message: update
Other:
- board size 100.5 x 82.5 mm -> 100 x 82.5 mm
Changed lines of the file:
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@@
 <board>
 <plain>
-<wire x1="66.167" y1="0" x2="66.167" y2="82.55" width="0" layer="20"/>
-<wire x1="-34.29" y1="0" x2="-34.29" y2="82.55" width="0" layer="20"/>
-<wire x1="-34.29" y1="82.55" x2="6.731" y2="82.55" width="0" layer="20"/>
-<wire x1="8.636" y1="82.55" x2="66.167" y2="82.55" width="0" layer="20"/>
-<wire x1="66.167" y1="0" x2="-34.29" y2="0" width="0" layer="20"/>
+<wire x1="65.8" y1="0" x2="65.8" y2="82.55" width="0" layer="20"/>
+<wire x1="-34.19" y1="0" x2="-34.19" y2="82.55" width="0" layer="20"/>
+<wire x1="-34.19" y1="82.55" x2="6.731" y2="82.55" width="0" layer="20"/>
+<wire x1="8.636" y1="82.55" x2="65.8" y2="82.55" width="0" layer="20"/>
+<wire x1="65.8" y1="0" x2="-34.19" y2="0" width="0" layer="20"/>
 <wire x1="6.731" y1="82.55" x2="6.731" y2="74.93" width="0" layer="20"/>
 <wire x1="6.731" y1="74.93" x2="8.636" y2="74.93" width="0" layer="20"/>
